Commit message: Chapter 7 Code

File: Chapter3/mastering_ros_robot_description_pkg/urdf/seven_dof_arm_with_rgbd.xacro (robot description, xacro)
@@ -373,6 +373,6 @@
   <!-- Define RGB-D sensor -->
   <xacro:xtion_pro_live name="rgbd_camera" parent="base">
-    <origin xyz="0.15 0.0 0.8" rpy="0 ${75.0 * deg_to_rad} 0"/>
-    <optical_origin xyz="0 0 0" rpy="${-90.0 * deg_to_rad} 0 ${-90.0 * deg_to_rad}"/>
+    <origin xyz="0.1 0.0 0.9" rpy="${0.0 * deg_to_rad} ${70.0 * deg_to_rad} ${0.0 * deg_to_rad}"/>
+    <origin xyz="0 0 0" rpy="${-90 * deg_to_rad} ${0 * deg_to_rad} ${-90 * deg_to_rad}" />
   </xacro:xtion_pro_live>
 	<!-- Transmissions for ROS Control -->
